File: JLCPCB-4Layer/JLCPCB-4Layer.kicad_pcb (KiCad board)
At the start: 4 copper layers, 0 parts

Commit message: huge whack of updates across the board
Other:
- net class Default removed
- net class JLC2313-84R-CLR removed
- net class JLC2313-84R-PCIe removed
- net class JLC2313-90R-RefClk removed
- net class POWER removed
- net class USB_D removed
- net class VCC removed
- net class VIN removed
Changed lines of the file:
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@@
-(kicad_pcb (version 20171130) (host pcbnew "(5.1.2-201-g3c8f901a1)")
+(kicad_pcb (version 20211014) (generator pcbnew)
   (general
     (thickness 1.6002)
-    (drawings 0)
-    (tracks 0)
-    (zones 0)
-    (modules 0)
-    (nets 1)
   )
-  (page A4)
+  (paper "A4")
   (title_block
-    (rev 1)
+    (rev "1")
   )
   (layers
-    (0 F.Cu signal)
-    (1 In1.Cu power)
-    (2 In2.Cu power)
-    (31 B.Cu signal)
-    (32 B.Adhes user)
-    (33 F.Adhes user)
-    (34 B.Paste user)
-    (35 F.Paste user)
-    (36 B.SilkS user)
-    (37 F.SilkS user)
-    (38 B.Mask user)
-    (39 F.Mask user)
-    (40 Dwgs.User user hide)
-    (41 Cmts.User user hide)
-    (42 Eco1.User user)
-    (43 Eco2.User user)
-    (44 Edge.Cuts user)
-    (45 Margin user)
-    (46 B.CrtYd user)
-    (47 F.CrtYd user)
-    (48 B.Fab user hide)
-    (49 F.Fab user)
+    (0 "F.Cu" signal)
+    (1 "In1.Cu" power)
+    (2 "In2.Cu" power)
+    (31 "B.Cu" signal)
+    (32 "B.Adhes" user "B.Adhesive")
+    (33 "F.Adhes" user "F.Adhesive")
+    (34 "B.Paste" user)
+    (35 "F.Paste" user)
+    (36 "B.SilkS" user "B.Silkscreen")
+    (37 "F.SilkS" user "F.Silkscreen")
+    (38 "B.Mask" user)
+    (39 "F.Mask" user)
+    (40 "Dwgs.User" user "User.Drawings")
+    (41 "Cmts.User" user "User.Comments")
+    (42 "Eco1.User" user "User.Eco1")
+    (43 "Eco2.User" user "User.Eco2")
+    (44 "Edge.Cuts" user)
+    (45 "Margin" user)
+    (46 "B.CrtYd" user "B.Courtyard")
+    (47 "F.CrtYd" user "F.Courtyard")
+    (48 "B.Fab" user)
+    (49 "F.Fab" user)
   )
   (setup
-    (last_trace_width 0.127)
-    (user_trace_width 0.127)
-    (user_trace_width 0.1524)
-    (user_trace_width 0.254)
-    (user_trace_width 0.3175)
-    (user_trace_width 0.381)
-    (user_trace_width 0.508)
-    (trace_clearance 0.127)
-    (zone_clearance 0.1524)
-    (zone_45_only yes)
-    (trace_min 0.127)
-    (via_size 0.45)
-    (via_drill 0.2)
-    (via_min_size 0.45)
-    (via_min_drill 0.2)
-    (user_via 0.45 0.2)
-    (user_via 0.6 0.3)
-    (user_via 0.8 0.4)
-    (uvia_size 0.6)
-    (uvia_drill 0.3)
-    (uvias_allowed no)
-    (uvia_min_size 0.45)
-    (uvia_min_drill 0.2)
-    (edge_width 0.05)
-    (segment_width 0.254)
-    (pcb_text_width 0.254)
-    (pcb_text_size 1.524 1.524)
-    (mod_edge_width 0.127)
-    (mod_text_size 0.8 0.8)
-    (mod_text_width 0.1524)
-    (pad_size 1.524 1.524)
-    (pad_drill 0.762)
     (pad_to_mask_clearance 0)
     (solder_mask_min_width 0.12)
-    (aux_axis_origin 0 0)
-    (visible_elements 7FFFFFFF)
     (pcbplotparams
-      (layerselection 0x010fc_ffffffff)
+      (layerselection 0x00010fc_ffffffff)
+      (disableapertmacros false)
       (usegerberextensions false)
       (usegerberattributes false)
       (usegerberadvancedattributes false)
       (creategerberjobfile false)
+      (svguseinch false)
+      (svgprecision 6)
       (excludeedgelayer true)
-      (linewidth 0.152400)
       (plotframeref false)
       (viasonmask false)
@@
       (hpglpenspeed 20)
       (hpglpendiameter 15.000000)
+      (dxfpolygonmode true)
+      (dxfimperialunits true)
+      (dxfusepcbnewfont true)
       (psnegative false)
       (psa4output false)
@@
       (plotvalue false)
       (plotinvisibletext false)
-      (padsonsilk false)
+      (sketchpadsonfab false)
       (subtractmaskfromsilk true)
       (outputformat 1)
@@
       (drillshape 0)
       (scaleselection 1)
-      (outputdirectory "./gerbers"))
+      (outputdirectory "./gerbers")
+    )
   )
   (net 0 "")
-  (net_class Default "This is the default net class."
-    (clearance 0.127)
-    (trace_width 0.127)
-    (via_dia 0.6)
-    (via_drill 0.3)
-    (uvia_dia 0.6858)
-    (uvia_drill 0.3302)
-    (diff_pair_width 0.1524)
-    (diff_pair_gap 0.127)
-  )
-  (net_class USB_D ""
-    (clearance 0.1524)
-    (trace_width 0.1524)
-    (via_dia 0.6)
-    (via_drill 0.3)
-    (uvia_dia 0.6858)
-    (uvia_drill 0.3302)
-    (diff_pair_width 0.1524)
-    (diff_pair_gap 0.1524)
-  )
-  (net_class VCC ""
-    (clearance 0.127)
-    (trace_width 0.2)
-    (via_dia 0.6)
-    (via_drill 0.3)
-    (uvia_dia 0.6858)
-    (uvia_drill 0.3302)
-    (diff_pair_width 0.1524)
-    (diff_pair_gap 0.254)
-  )
-  (net_class VIN ""
-    (clearance 0.254)
-    (trace_width 0.4)
-    (via_dia 0.8)
-    (via_drill 0.4)
-    (uvia_dia 0.6858)
-    (uvia_drill 0.3302)
-    (diff_pair_width 0.1524)
-    (diff_pair_gap 0.127)
-  )
-    (net_class JLC2313-84R-CLR ""
-    (clearance 0.75)
-    (trace_width 0.15635)
-    (via_dia 0.45)
-    (via_drill 0.2)
-    (uvia_dia 0.3)
-    (uvia_drill 0.1)
-    (diff_pair_width 0.15635)
-    (diff_pair_gap 0.127)
-  )
-  (net_class JLC2313-84R-PCIe ""
-    (clearance 0.127)
-    (trace_width 0.15635)
-    (via_dia 0.45)
-    (via_drill 0.2)
-    (uvia_dia 0.3)
-    (uvia_drill 0.1)
-    (diff_pair_width 0.15635)
-    (diff_pair_gap 0.127)
-  )
-  (net_class JLC2313-90R-RefClk ""
-    (clearance 0.127)
-    (trace_width 0.13422)
-    (via_dia 0.45)
-    (via_drill 0.2)
-    (uvia_dia 0.3)
-    (uvia_drill 0.1)
-    (diff_pair_width 0.13422)
-    (diff_pair_gap 0.127)
-  )
-  (net_class POWER ""
-    (clearance 0.127)
-    (trace_width 0.381)
-    (via_dia 0.6)
-    (via_drill 0.3)
-    (uvia_dia 0.6)
-    (uvia_drill 0.1)
-    (diff_pair_width 0.381)
-    (diff_pair_gap 0.127)
-  )
 )
